Commit message: video n02

File: urdf/mrm.xacro (robot description, xacro)
@@ -1,26 +1,47 @@
 <?xml version="1.0" ?>
 <robot name="mrm" xmlns:xacro="http://www.ros.org/wiki/xacro">
-    <link name="base_link">
-        <visual>
-          <origin rpy="0 0 0" xyz="0 0 0" />
-          <geometry>
-            <box size="1 1 1" />
-          </geometry>
-        </visual>
-    </link>
-      <joint name="base_link__link_01" type="revolute">
-        <axis xyz="0 0 1"/>
-        <limit effort="1000.0" lower="-3.14" upper="3.14" velocity="0.5"/>
-        <origin rpy="0 0 0" xyz="0 0 0.5"/>
-        <parent link="base_link"/>
-        <child link="link_01"/>
-      </joint>
-    <link name="link_01">
-        <visual>
-          <origin rpy="0 0 0" xyz="0 0 0.2" />
-          <geometry>
-            <cylinder radius="0.35" length="0.4" />
-          </geometry>
-        </visual>
-    </link>
+  <!-- BGN - Include -->
+  <xacro:include filename="$(find mrm_description)/urdf/robot_parameters.xacro" />
+  <xacro:include filename="$(find mrm_description)/urdf/links_joints.xacro" />
+  <!-- END - Include -->
+  <!-- BGN - Robot description -->
+  <m_link_box name="${link_00_name}"
+              origin_rpy="0 0 0" origin_xyz="0 0 0"
+              size="1 1 1" />
+  <m_joint name="${link_00_name}__${link_01_name}" type="revolute"
+           axis_xyz="0 0 1"
+           origin_rpy="0 0 0" origin_xyz="0 0 0.5"
+           parent="base_link" child="link_01" />
+  <m_link_cylinder name="${link_01_name}"
+              origin_rpy="0 0 0" origin_xyz="0 0 0.2"
+              length="0.4" radius="0.35" />
+  <m_joint name="${link_01_name}__${link_02_name}" type="revolute"
+           axis_xyz="0 1 0"
+           origin_rpy="0 0 0" origin_xyz="0 0 0.4"
+           parent="link_01" child="link_02" />
+  <m_link_cylinder name="${link_02_name}"
+              origin_rpy="0 0 0" origin_xyz="0 0 0.4"
+              radius="0.15" length="0.8" />
+  <m_joint name="${link_02_name}__${link_03_name}" type="revolute"
+           axis_xyz="0 1 0"
+           origin_rpy="0 0 0" origin_xyz="0 0 0.8"
+           parent="link_02" child="link_03" />
+  <m_link_cylinder name="${link_03_name}"
+              origin_rpy="0 0 0" origin_xyz="0 0 0.4"
+              radius="0.15" length="0.8" />
+  <m_joint name="${link_03_name}__${link_04_name}" type="revolute"
+           axis_xyz="0 1 0"
+           origin_rpy="0 0 0" origin_xyz="0 0 0.8"
+           parent="link_03" child="link_04" />
+  <m_link_cylinder name="${link_04_name}"
+              origin_rpy="0 0 0" origin_xyz="0 0 0.4"
+              radius="0.15" length="0.8" />
+  <m_joint name="${link_04_name}__${link_05_name}" type="revolute"
+           axis_xyz="0 0 1"
+           origin_rpy="0 0 0" origin_xyz="0 0 0.8"
+           parent="link_04" child="link_05" />
+  <m_link_cylinder name="${link_05_name}"
+              origin_rpy="0 0 0" origin_xyz="0 0 0.125"
+              radius="0.15" length="0.25" />
+  <!-- END - Robot description -->
 </robot>

Commit message: video n04 - controllers to simplified model

File: urdf/mrm.xacro (robot description, xacro)
@@ -8,4 +8,8 @@
   <m_link_box name="${link_00_name}"
               origin_rpy="0 0 0" origin_xyz="0 0 0"
+              mass="1024"
+              ixx="170.667" ixy="0" ixz="0"
+              iyy="170.667" iyz="0"
+              izz="170.667"
               size="1 1 1" />
   <m_joint name="${link_00_name}__${link_01_name}" type="revolute"
@@ -13,6 +17,20 @@
            origin_rpy="0 0 0" origin_xyz="0 0 0.5"
            parent="base_link" child="link_01" />
+  <transmission name="trans_${link_00_name}__${link_01_name}">
+    <type>transmission_interface/SimpleTransmission</type>
+    <joint name="${link_00_name}__${link_01_name}">
+      <hardwareInterface>hardware_interface/EffortJointInterface</hardwareInterface>
+    </joint>
+    <actuator name="motor_${link_00_name}__${link_01_name}">
+      <hardwareInterface>hardware_interface/EffortJointInterface</hardwareInterface>
+      <mechanicalReduction>1</mechanicalReduction>
+    </actuator>
+  </transmission>
   <m_link_cylinder name="${link_01_name}"
               origin_rpy="0 0 0" origin_xyz="0 0 0.2"
+              mass="157.633"
+              ixx="13.235" ixy="0" ixz="0"
+              iyy="13.235" iyz="0"
+              izz="9.655"
               length="0.4" radius="0.35" />
   <m_joint name="${link_01_name}__${link_02_name}" type="revolute"
@@ -20,7 +38,22 @@
            origin_rpy="0 0 0" origin_xyz="0 0 0.4"
            parent="link_01" child="link_02" />
+  <transmission name="trans_${link_01_name}__${link_02_name}">
+    <type>transmission_interface/SimpleTransmission</type>
+    <joint name="${link_01_name}__${link_02_name}">
+      <hardwareInterface>hardware_interface/EffortJointInterface</hardwareInterface>
+    </joint>
+    <actuator name="motor_${link_01_name}__${link_02_name}">
+      <hardwareInterface>hardware_interface/EffortJointInterface</hardwareInterface>
+      <mechanicalReduction>1</mechanicalReduction>
+    </actuator>
+  </transmission>
   <m_link_cylinder name="${link_02_name}"
               origin_rpy="0 0 0" origin_xyz="0 0 0.4"
+              mass="57.906"
+              ixx="12.679" ixy="0" ixz="0"
+              iyy="12.679" iyz="0"
+              izz="0.651"
               radius="0.15" length="0.8" />
+  <!--
   <m_joint name="${link_02_name}__${link_03_name}" type="revolute"
            axis_xyz="0 1 0"
@@ -29,4 +62,8 @@
   <m_link_cylinder name="${link_03_name}"
               origin_rpy="0 0 0" origin_xyz="0 0 0.4"
+              mass="57.906"
+              ixx="12.679" ixy="0" ixz="0"
+              iyy="12.679" iyz="0"
+              izz="0.651"
               radius="0.15" length="0.8" />
   <m_joint name="${link_03_name}__${link_04_name}" type="revolute"
@@ -36,4 +73,8 @@
   <m_link_cylinder name="${link_04_name}"
               origin_rpy="0 0 0" origin_xyz="0 0 0.4"
+              mass="57.906"
+              ixx="12.679" ixy="0" ixz="0"
+              iyy="12.679" iyz="0"
+              izz="0.651"
               radius="0.15" length="0.8" />
   <m_joint name="${link_04_name}__${link_05_name}" type="revolute"
@@ -43,5 +84,14 @@
   <m_link_cylinder name="${link_05_name}"
               origin_rpy="0 0 0" origin_xyz="0 0 0.125"
+              mass="18.056"
+              ixx="0.479" ixy="0" ixz="0"
+              iyy="0.479" iyz="0"
+              izz="0.204"
               radius="0.15" length="0.25" />
+  -->
   <!-- END - Robot description -->
+  <gazebo>
+    <plugin name="gazebo_ros_control" filename="libgazebo_ros_control.so">
+    </plugin>
+  </gazebo>
 </robot>
